Commit message: fix tests for multiple trees, and clean up regression tests
--HG--
extra : convert_revision : svn%3Aeb33c2ac-9c88-4c90-87e0-44a10359b0c3/stacks/robot_model/trunk%4028628

File: urdf/test/pr2_desc_no_joint.urdf (robot description, URDF)
Before this commit: robot pr2, 1 links, 1 joints
Joints:
- joint fl_caster_rotation_joint: type None -> continuous
