Commit message: minor change, base_laser --> base_laser_link link name update in test xmls.
--HG--
extra : convert_revision : svn%3Aeb33c2ac-9c88-4c90-87e0-44a10359b0c3/stacks/robot_model/trunk%4025915

File: robot_state_publisher/test/pr2.urdf (robot description, URDF)
Before this commit: robot pr2, 71 links, 73 joints
Links:
- removed link base_laser
- added link base_laser_link, mass 1.0; collision box size=0.06 0.06 0.03; visual box size=0.06 0.06 0.03
Joints:
- joint base_laser_joint: child base_laser -> base_laser_link

Commit message: Add regression tests for cases with 1, 2 links in urdf, with and without fixed joints. Fix bug where 2-link urdf is not accepted #4042 #4185
--HG--
extra : convert_revision : svn%3Aeb33c2ac-9c88-4c90-87e0-44a10359b0c3/stacks/robot_model/trunk%4030389

File: robot_state_publisher/test/pr2.urdf (robot description, URDF)
Before this commit: robot pr2, 71 links, 73 joints
Links:
- removed link l_gripper_float_link
- removed link narrow_stereo_l_stereo_camera_frame
- removed link narrow_stereo_r_stereo_camera_frame
- removed link plug_holder
- removed link r_gripper_float_link
- removed link wide_stereo_l_stereo_camera_frame
- removed link wide_stereo_r_stereo_camera_frame
- added link base_footprint, mass 1.0; collision box size=0.001 0.001 0.001; visual box size=0.01 0.01 0.01
- added link imu_link, mass 0.001; collision box size=.001 .001 .001; visual box size=0.001 0.001 0.001
- added link l_gripper_l_parallel_link, mass 0.17126; collision box size=0.0914942479 0.005 0.005
- added link l_gripper_led_frame
- added link l_gripper_r_parallel_link, mass 0.17389; collision box size=0.0914942479 0.005 0.005
- added link narrow_stereo_gazebo_l_stereo_camera_frame, mass 0.01; collision box size=0.01 0.01 0.01; visual box size=0.01 0.01 0.01
- added link narrow_stereo_gazebo_l_stereo_camera_optical_frame
- added link narrow_stereo_gazebo_r_stereo_camera_frame, mass 0.01; collision box size=0.01 0.01 0.01; visual box size=0.01 0.01 0.01
- added link narrow_stereo_gazebo_r_stereo_camera_optical_frame
- added link r_gripper_l_parallel_link, mass 0.17126; collision box size=0.0914942479 0.005 0.005
- added link r_gripper_led_frame
- added link r_gripper_r_parallel_link, mass 0.17389; collision box size=0.0914942479 0.005 0.005
- added link wide_stereo_gazebo_l_stereo_camera_frame, mass 0.01; collision box size=0.01 0.01 0.01; visual box size=0.01 0.01 0.01
- added link wide_stereo_gazebo_l_stereo_camera_optical_frame
- added link wide_stereo_gazebo_r_stereo_camera_frame, mass 0.01; collision box size=0.01 0.01 0.01; visual box size=0.01 0.01 0.01
- added link wide_stereo_gazebo_r_stereo_camera_optical_frame
- link base_laser_link: mass 1.0 -> 0.001; geometry collision box size=.001 .001 .001; visual box size=0.001 0.001 0.001
- link base_link: geometry collision mesh filename=package://pr2_description/meshes/base_v0/base_L.stl; visual mesh filename=package://pr2_description/meshes/base_v0/base.stl
- link bl_caster_l_wheel_link: geometry collision cylinder length=0.034 radius=0.074792; visual mesh filename=package://pr2_description/meshes/base_v0/wheel.stl
- link bl_caster_r_wheel_link: geometry collision cylinder length=0.034 radius=0.074792; visual mesh filename=package://pr2_description/meshes/base_v0/wheel.stl
- link bl_caster_rotation_link: geometry collision mesh filename=package://pr2_description/meshes/base_v0/caster_L.stl; visual mesh filename=package://pr2_description/meshes/base_v0/caster.stl
- link br_caster_l_wheel_link: geometry collision cylinder length=0.034 radius=0.074792; visual mesh filename=package://pr2_description/meshes/base_v0/wheel.stl
- link br_caster_r_wheel_link: geometry collision cylinder length=0.034 radius=0.074792; visual mesh filename=package://pr2_description/meshes/base_v0/wheel.stl
- link br_caster_rotation_link: geometry collision mesh filename=package://pr2_description/meshes/base_v0/caster_L.stl; visual mesh filename=package://pr2_description/meshes/base_v0/caster.stl
- link double_stereo_link: geometry collision box size=0.02 0.12 0.05; visual box size=0.02 0.12 0.05
- link fl_caster_l_wheel_link: geometry collision cylinder length=0.034 radius=0.074792; visual mesh filename=package://pr2_description/meshes/base_v0/wheel.stl
- link fl_caster_r_wheel_link: geometry collision cylinder length=0.034 radius=0.074792; visual mesh filename=package://pr2_description/meshes/base_v0/wheel.stl
- link fl_caster_rotation_link: geometry collision mesh filename=package://pr2_description/meshes/base_v0/caster_L.stl; visual mesh filename=package://pr2_description/meshes/base_v0/caster.stl
- link fr_caster_l_wheel_link: geometry collision cylinder length=0.034 radius=0.074792; visual mesh filename=package://pr2_description/meshes/base_v0/wheel.stl
- link fr_caster_r_wheel_link: geometry collision cylinder length=0.034 radius=0.074792; visual mesh filename=package://pr2_description/meshes/base_v0/wheel.stl
- link fr_caster_rotation_link: geometry collision mesh filename=package://pr2_description/meshes/base_v0/caster_L.stl; visual mesh filename=package://pr2_description/meshes/base_v0/caster.stl
- link head_pan_link: geometry collision mesh filename=package://pr2_description/meshes/head_v0/head_pan_L.stl; visual mesh filename=package://pr2_description/meshes/head_v0/head_pan.stl
- link head_tilt_link: geometry collision mesh filename=package://pr2_description/meshes/head_v0/head_tilt_L.stl; visual mesh filename=package://pr2_description/meshes/head_v0/head_tilt.stl
- link high_def_frame: geometry collision box size=0.01 0.01 0.01; visual box size=0.04 0.04 0.04
- link high_def_optical_frame: geometry collision box size=0.01 0.01 0.01; visual cylinder length=0.05 radius=0.02
- link l_elbow_flex_link: geometry collision mesh filename=package://pr2_description/meshes/upper_arm_v0/elbow_flex.stl; visual mesh filename=package://pr2_description/meshes/upper_arm_v0/elbow_flex.stl
- link l_forearm_cam_optical_frame: mass 0.01 -> None; geometry 
- link l_forearm_link: geometry collision mesh filename=package://pr2_description/meshes/forearm_v0/forearm.stl; visual mesh filename=package://pr2_description/meshes/forearm_v0/forearm.stl
- link l_forearm_roll_link: geometry collision mesh filename=package://pr2_description/meshes/upper_arm_v0/forearm_roll_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; visual mesh filename=package://pr2_description/meshes/upper_arm_v0/forearm_roll.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
- link l_gripper_l_finger_link: geometry collision mesh filename=package://pr2_description/meshes/gripper_v0/l_finger.stl; visual mesh filename=package://pr2_description/meshes/gripper_v0/l_finger.stl
- link l_gripper_l_finger_tip_link: geometry collision mesh filename=package://pr2_description/meshes/gripper_v0/l_finger_tip.stl; visual mesh filename=package://pr2_description/meshes/gripper_v0/l_finger_tip.stl
- link l_gripper_palm_link: geometry collision mesh filename=package://pr2_description/meshes/gripper_v0/gripper_palm.stl; visual mesh filename=package://pr2_description/meshes/gripper_v0/gripper_palm.stl
- link l_gripper_r_finger_link: geometry collision mesh filename=package://pr2_description/meshes/gripper_v0/l_finger.stl; visual mesh filename=package://pr2_description/meshes/gripper_v0/l_finger.stl
- link l_gripper_r_finger_tip_link: geometry collision mesh filename=package://pr2_description/meshes/gripper_v0/l_finger_tip.stl; visual mesh filename=package://pr2_description/meshes/gripper_v0/l_finger_tip.stl
- link l_gripper_tool_frame: mass 0.01 -> None; geometry 
- link l_shoulder_lift_link: geometry collision mesh filename=package://pr2_description/meshes/shoulder_v0/shoulder_lift.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; visual mesh filename=package://pr2_description/meshes/shoulder_v0/shoulder_lift.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
- link l_shoulder_pan_link: geometry collision mesh filename=package://pr2_description/meshes/shoulder_v0/shoulder_pan.s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; visual mesh filename=package://pr2_description/meshes/shoulder_v0/shoulder_pan.s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
- link l_upper_arm_link: geometry collision mesh filename=package://pr2_description/meshes/upper_arm_v0/upper_arm.stl; visual mesh filename=package://pr2_description/meshes/upper_arm_v0/upper_arm.stl
- link l_upper_arm_roll_link: geometry collision mesh filename=package://pr2_description/meshes/shoulder_v0/upper_arm_roll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; visual mesh filename=package://pr2_description/meshes/shoulder_v0/upper_arm_roll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
- link l_wrist_flex_link: geometry collision mesh filename=package://pr2_description/meshes/forearm_v0/wrist_flex.stl; visual mesh filename=package://pr2_description/meshes/forearm_v0/wrist_flex.stl
- link l_wrist_roll_link: geometry collision mesh filename=package://pr2_description/meshes/forearm_v0/wrist_roll_L.stl; visual mesh filename=package://pr2_description/meshes/forearm_v0/wrist_roll.stl
- link laser_tilt_mount_link: geometry collision mesh filename=package://pr2_description/meshes/tilting_laser_v0/tilting_h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; visual mesh filename=package://pr2_description/meshes/tilting_laser_v0/tilting_h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
- link narrow_stereo_link: geometry collision box size=0.001 0.001 0.001; visual box size=0.001 0.001 0.001
- link narrow_stereo_optical_frame: mass 0.01 -> None; geometry 
- link r_elbow_flex_link: geometry collision mesh filename=package://pr2_description/meshes/upper_arm_v0/elbow_flex.stl; visual mesh filename=package://pr2_description/meshes/upper_arm_v0/elbow_flex.stl
- link r_forearm_cam_optical_frame: mass 0.01 -> None; geometry 
- link r_forearm_link: geometry collision mesh filename=package://pr2_description/meshes/forearm_v0/forearm.stl; visual mesh filename=package://pr2_description/meshes/forearm_v0/forearm.stl
- link r_forearm_roll_link: geometry collision mesh filename=package://pr2_description/meshes/upper_arm_v0/forearm_roll_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; visual mesh filename=package://pr2_description/meshes/upper_arm_v0/forearm_roll.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
- link r_gripper_l_finger_link: geometry collision mesh filename=package://pr2_description/meshes/gripper_v0/l_finger.stl; visual mesh filename=package://pr2_description/meshes/gripper_v0/l_finger.stl
- link r_gripper_l_finger_tip_link: geometry collision mesh filename=package://pr2_description/meshes/gripper_v0/l_finger_tip.stl; visual mesh filename=package://pr2_description/meshes/gripper_v0/l_finger_tip.stl
- link r_gripper_palm_link: geometry collision mesh filename=package://pr2_description/meshes/gripper_v0/gripper_palm.stl; visual mesh filename=package://pr2_description/meshes/gripper_v0/gripper_palm.stl
- link r_gripper_r_finger_link: geometry collision mesh filename=package://pr2_description/meshes/gripper_v0/l_finger.stl; visual mesh filename=package://pr2_description/meshes/gripper_v0/l_finger.stl
- link r_gripper_r_finger_tip_link: geometry collision mesh filename=package://pr2_description/meshes/gripper_v0/l_finger_tip.stl; visual mesh filename=package://pr2_description/meshes/gripper_v0/l_finger_tip.stl
- link r_gripper_tool_frame: mass 0.01 -> None; geometry 
- link r_shoulder_lift_link: geometry collision mesh filename=package://pr2_description/meshes/shoulder_v0/shoulder_lift.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; visual mesh filename=package://pr2_description/meshes/shoulder_v0/shoulder_lift.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
- link r_shoulder_pan_link: geometry collision mesh filename=package://pr2_description/meshes/shoulder_v0/shoulder_pan.s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; visual mesh filename=package://pr2_description/meshes/shoulder_v0/shoulder_pan.s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
- link r_upper_arm_link: geometry collision mesh filename=package://pr2_description/meshes/upper_arm_v0/upper_arm.stl; visual mesh filename=package://pr2_description/meshes/upper_arm_v0/upper_arm.stl
- link r_upper_arm_roll_link: geometry collision mesh filename=package://pr2_description/meshes/shoulder_v0/upper_arm_roll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; visual mesh filename=package://pr2_description/meshes/shoulder_v0/upper_arm_roll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
- link r_wrist_flex_link: geometry collision mesh filename=package://pr2_description/meshes/forearm_v0/wrist_flex.stl; visual mesh filename=package://pr2_description/meshes/forearm_v0/wrist_flex.stl
- link r_wrist_roll_link: geometry collision mesh filename=package://pr2_description/meshes/forearm_v0/wrist_roll_L.stl; visual mesh filename=package://pr2_description/meshes/forearm_v0/wrist_roll.stl
- link torso_lift_link: geometry collision mesh filename=package://pr2_description/meshes/torso_v0/torso_lift_L.stl; visual mesh filename=package://pr2_description/meshes/torso_v0/torso_lift.stl
- link wide_stereo_link: geometry collision box size=0.001 0.001 0.001; visual box size=0.001 0.001 0.001
- link wide_stereo_optical_frame: mass 0.01 -> None; geometry 
Joints:
- removed joint base_joint
- removed joint l_gripper_float_joint
- removed joint narrow_stereo_l_stereo_camera_frame_joint
- removed joint narrow_stereo_r_stereo_camera_frame_joint
- removed joint plug_holder_joint
- removed joint r_gripper_float_joint
- removed joint wide_stereo_l_stereo_camera_frame_joint
- removed joint wide_stereo_r_stereo_camera_frame_joint
- added joint base_footprint_joint: type fixed, parent base_footprint, child base_link, origin xyz=0 0 0.051 rpy=0 0 0
- added joint imu_joint: type fixed, parent torso_lift_link, child imu_link, origin xyz=-0.02977 -0.1497 0.164 rpy=0 3.14159265359 0, axis 0 1 0
- added joint l_gripper_l_parallel_root_joint: type revolute, parent l_gripper_palm_link, child l_gripper_l_parallel_link, origin xyz=0.05891 0.031 0 rpy=0 0 0, axis 0 0 1, limit lower=0.0 upper=0.548 effort=1000.0 velocity=0.5, mimic joint=l_gripper_l_finger_joint multiplier=1 offset=0
- added joint l_gripper_led_joint: type fixed, parent l_gripper_palm_link, child l_gripper_led_frame, origin xyz=0.0513 0.0 .0244
- added joint l_gripper_r_parallel_root_joint: type revolute, parent l_gripper_palm_link, child l_gripper_r_parallel_link, origin xyz=0.05891 -0.031 0 rpy=0 0 0, axis 0 0 -1, limit lower=0.0 upper=0.548 effort=1000.0 velocity=0.5, mimic joint=l_gripper_l_finger_joint multiplier=-1 offset=0
- added joint narrow_stereo_gazebo_l_stereo_camera_frame_joint: type fixed, parent narrow_stereo_link, child narrow_stereo_gazebo_l_stereo_camera_frame, origin xyz=0 0 0 rpy=0 0 0
- added joint narrow_stereo_gazebo_l_stereo_camera_optical_frame_joint: type fixed, parent narrow_stereo_gazebo_l_stereo_camera_frame, child narrow_stereo_gazebo_l_stereo_camera_optical_frame, origin xyz=0 0 0 rpy=-1.57079632679 0.0 -1.57079632679
- added joint narrow_stereo_gazebo_r_stereo_camera_frame_joint: type fixed, parent narrow_stereo_gazebo_l_stereo_camera_frame, child narrow_stereo_gazebo_r_stereo_camera_frame, origin xyz=0.0 -0.09 0.0 rpy=0.0 0.0 0.0
- added joint narrow_stereo_gazebo_r_stereo_camera_optical_frame_joint: type fixed, parent narrow_stereo_gazebo_r_stereo_camera_frame, child narrow_stereo_gazebo_r_stereo_camera_optical_frame, origin xyz=0 0 0 rpy=-1.57079632679 0.0 -1.57079632679
- added joint r_gripper_l_parallel_root_joint: type revolute, parent r_gripper_palm_link, child r_gripper_l_parallel_link, origin xyz=0.05891 0.031 0 rpy=0 0 0, axis 0 0 1, limit lower=0.0 upper=0.548 effort=1000.0 velocity=0.5, mimic joint=r_gripper_l_finger_joint multiplier=1 offset=0
- added joint r_gripper_led_joint: type fixed, parent r_gripper_palm_link, child r_gripper_led_frame, origin xyz=0.0513 0.0 .0244
- added joint r_gripper_r_parallel_root_joint: type revolute, parent r_gripper_palm_link, child r_gripper_r_parallel_link, origin xyz=0.05891 -0.031 0 rpy=0 0 0, axis 0 0 -1, limit lower=0.0 upper=0.548 effort=1000.0 velocity=0.5, mimic joint=r_gripper_l_finger_joint multiplier=-1 offset=0
- added joint wide_stereo_gazebo_l_stereo_camera_frame_joint: type fixed, parent wide_stereo_link, child wide_stereo_gazebo_l_stereo_camera_frame, origin xyz=0 0 0 rpy=0 0 0
- added joint wide_stereo_gazebo_l_stereo_camera_optical_frame_joint: type fixed, parent wide_stereo_gazebo_l_stereo_camera_frame, child wide_stereo_gazebo_l_stereo_camera_optical_frame, origin xyz=0 0 0 rpy=-1.57079632679 0.0 -1.57079632679
- added joint wide_stereo_gazebo_r_stereo_camera_frame_joint: type fixed, parent wide_stereo_gazebo_l_stereo_camera_frame, child wide_stereo_gazebo_r_stereo_camera_frame, origin xyz=0.0 -0.09 0.0 rpy=0.0 0.0 0.0
- added joint wide_stereo_gazebo_r_stereo_camera_optical_frame_joint: type fixed, parent wide_stereo_gazebo_r_stereo_camera_frame, child wide_stereo_gazebo_r_stereo_camera_optical_frame, origin xyz=0 0 0 rpy=-1.57079632679 0.0 -1.57079632679
- joint base_laser_joint: axis (none) -> 0 1 0
- joint bl_caster_rotation_joint: origin xyz=-0.2225 0.2225 0.0282 rpy=0 0 0 -> xyz=-0.2246 0.2246 0.0282 rpy=0 0 0
- joint br_caster_rotation_joint: origin xyz=-0.2225 -0.2225 0.0282 rpy=0 0 0 -> xyz=-0.2246 -0.2246 0.0282 rpy=0 0 0
- joint fl_caster_rotation_joint: origin xyz=0.2225 0.2225 0.0282 rpy=0 0 0 -> xyz=0.2246 0.2246 0.0282 rpy=0 0 0
- joint fr_caster_rotation_joint: origin xyz=0.2225 -0.2225 0.0282 rpy=0 0 0 -> xyz=0.2246 -0.2246 0.0282 rpy=0 0 0
- joint head_pan_joint: limit lower=-2.92 upper=2.92 effort=2.645 velocity=6 -> lower=-3.007 upper=3.007 effort=2.645 velocity=6; origin xyz=0.0    0.0     0.3915 rpy=0.0 0.0 0.0 -> xyz=-0.01707 0.0 0.38145 rpy=0.0 0.0 0.0
- joint head_tilt_joint: limit lower=-0.55 upper=1.047 effort=12.21 velocity=100 -> lower=-0.471238 upper=1.39626 effort=15 velocity=5; origin xyz=0.058 0 0 rpy=0 0 0 -> xyz=0.068 0 0 rpy=0 0 0
- joint l_elbow_flex_joint: limit lower=-2.3 upper=0.1 effort=30 velocity=3.3 -> lower=-2.3213 upper=0.00 effort=30 velocity=3.3
- joint l_forearm_cam_frame_joint: origin xyz=.15 0 .07 rpy=1.57079632679 -0.785398163397 0 -> xyz=.135 0 .044 rpy=-1.57079632679 -0.562868683768 0
- joint l_forearm_roll_joint: axis -1 0 0 -> 1 0 0
- joint l_gripper_joint: axis 0 0 1 -> 0 1 0; limit lower=0.0 upper=0.09 effort=100.0 velocity=0.2 -> lower=0.0 upper=0.09 effort=1000.0 velocity=0.2
- joint l_gripper_l_finger_joint: limit lower=0.0 upper=0.548 effort=100.0 velocity=0.5 -> lower=0.0 upper=0.548 effort=1000.0 velocity=0.5
- joint l_gripper_l_finger_tip_joint: limit lower=0.0 upper=0.548 effort=100.0 velocity=0.5 -> lower=0.0 upper=0.548 effort=1000.0 velocity=0.5
- joint l_gripper_r_finger_joint: limit lower=0.0 upper=0.548 effort=100.0 velocity=0.5 -> lower=0.0 upper=0.548 effort=1000.0 velocity=0.5
- joint l_gripper_r_finger_tip_joint: limit lower=0.0 upper=0.548 effort=100.0 velocity=0.5 -> lower=0.0 upper=0.548 effort=1000.0 velocity=0.5
- joint l_wrist_flex_joint: axis 0 -1 0 -> 0 1 0; limit lower=-0.1 upper=2.2 effort=200 velocity=3.078 -> lower=-2.094 upper=0.0 effort=10 velocity=3.078; origin xyz=0.32025 0 0 rpy=0 0 0 -> xyz=0.321 0 0 rpy=0 0 0
- joint laser_tilt_mount_joint: limit lower=-0.785 upper=1.57 effort=0.5292 velocity=10.0 -> lower=-0.7854 upper=1.48353 effort=0.65 velocity=10.0; origin xyz=0.1 0 0.235 rpy=0 0 0 -> xyz=0.09893 0 0.227 rpy=0 0 0
- joint narrow_stereo_frame_joint: origin xyz=0 0.015 0 rpy=0 0 0 -> xyz=0.0 0.06 0.0305 rpy=0.0   0.0   0.0
- joint narrow_stereo_optical_frame_joint: origin xyz=0.0            0.045   0.0305 rpy=-1.57079632679 0.0 -1.57079632679 -> xyz=0 0 0 rpy=-1.57079632679 0.0 -1.57079632679
- joint r_elbow_flex_joint: limit lower=-2.3 upper=0.1 effort=30 velocity=3.3 -> lower=-2.3213 upper=0.00 effort=30 velocity=3.3
- joint r_forearm_cam_frame_joint: origin xyz=.15 0 .07 rpy=-1.57079632679 -0.785398163397 0 -> xyz=.135 0 .044 rpy=1.57079632679 -0.562868683768 0
- joint r_forearm_roll_joint: axis -1 0 0 -> 1 0 0
- joint r_gripper_joint: axis 0 0 1 -> 0 1 0; limit lower=0.0 upper=0.09 effort=100.0 velocity=0.2 -> lower=0.0 upper=0.09 effort=1000.0 velocity=0.2
- joint r_gripper_l_finger_joint: limit lower=0.0 upper=0.548 effort=100.0 velocity=0.5 -> lower=0.0 upper=0.548 effort=1000.0 velocity=0.5
- joint r_gripper_l_finger_tip_joint: limit lower=0.0 upper=0.548 effort=100.0 velocity=0.5 -> lower=0.0 upper=0.548 effort=1000.0 velocity=0.5
- joint r_gripper_r_finger_joint: limit lower=0.0 upper=0.548 effort=100.0 velocity=0.5 -> lower=0.0 upper=0.548 effort=1000.0 velocity=0.5
- joint r_gripper_r_finger_tip_joint: limit lower=0.0 upper=0.548 effort=100.0 velocity=0.5 -> lower=0.0 upper=0.548 effort=1000.0 velocity=0.5
- joint r_shoulder_pan_joint: origin xyz=0 -0.188 0.0 rpy=0 0 0 -> xyz=0.0 -0.188 0.0 rpy=0 0 0
- joint r_wrist_flex_joint: axis 0 -1 0 -> 0 1 0; limit lower=-0.1 upper=2.2 effort=200 velocity=3.078 -> lower=-2.094 upper=0.0 effort=10 velocity=3.078; origin xyz=0.32025 0 0 rpy=0 0 0 -> xyz=0.321 0 0 rpy=0 0 0
- joint torso_lift_joint: limit lower=0.0 upper=0.20 effort=10000 velocity=0.015 -> lower=0.0 upper=0.31 effort=10000 velocity=0.013
- joint wide_stereo_frame_joint: origin xyz=0 -0.015 0 rpy=0 0 0 -> xyz=0.0 0.03 0.0305 rpy=0.0   0.0   0.0
- joint wide_stereo_optical_frame_joint: origin xyz=0.0            0.045   0.0305 rpy=-1.57079632679 0.0 -1.57079632679 -> xyz=0 0 0 rpy=-1.57079632679 0.0 -1.57079632679
