Commit message: fix regression tests
--HG--
branch : robot_model-1.4
extra : convert_revision : svn%3Aeb33c2ac-9c88-4c90-87e0-44a10359b0c3/stacks/robot_model/branches/robot_model-1.4%4035062

File: robot_state_publisher/test/pr2.urdf (robot description, URDF)
Before this commit: robot pr2, 80 links, 81 joints
Links:
- removed link l_gripper_l_parallel_link
- removed link l_gripper_r_parallel_link
- removed link r_gripper_l_parallel_link
- removed link r_gripper_r_parallel_link
- added link base_bellow_link, mass 1.0; collision box size=0.05 0.37 0.3; visual box size=0.05 0.37 0.3
- added link l_gripper_l_finger_tip_frame
- added link l_torso_lift_side_plate_link, mass 0.1
- added link projector_wg6802418_child_frame, mass 0.01; collision box size=0.01 0.01 0.01; visual cylinder length=0.05 radius=0.02
- added link projector_wg6802418_frame, mass 0.01; collision box size=0.01 0.01 0.01; visual box size=0.04 0.04 0.04
- added link r_gripper_l_finger_tip_frame
- added link r_torso_lift_side_plate_link, mass 0.1
- link base_link: geometry collision mesh filename=package://pr2_description/meshes/base_v0/base_L.stl; visual mesh filename=package://pr2_description/meshes/base_v0/base.dae
- link bl_caster_l_wheel_link: geometry collision cylinder length=0.034 radius=0.074792; visual mesh filename=package://pr2_description/meshes/base_v0/wheel.dae
- link bl_caster_r_wheel_link: geometry collision cylinder length=0.034 radius=0.074792; visual mesh filename=package://pr2_description/meshes/base_v0/wheel.dae
- link br_caster_l_wheel_link: geometry collision cylinder length=0.034 radius=0.074792; visual mesh filename=package://pr2_description/meshes/base_v0/wheel.dae
- link br_caster_r_wheel_link: geometry collision cylinder length=0.034 radius=0.074792; visual mesh filename=package://pr2_description/meshes/base_v0/wheel.dae
- link double_stereo_link: geometry visual box size=0.02 0.12 0.05
- link fl_caster_l_wheel_link: geometry collision cylinder length=0.034 radius=0.074792; visual mesh filename=package://pr2_description/meshes/base_v0/wheel.dae
- link fl_caster_r_wheel_link: geometry collision cylinder length=0.034 radius=0.074792; visual mesh filename=package://pr2_description/meshes/base_v0/wheel.dae
- link fr_caster_l_wheel_link: geometry collision cylinder length=0.034 radius=0.074792; visual mesh filename=package://pr2_description/meshes/base_v0/wheel.dae
- link fr_caster_r_wheel_link: geometry collision cylinder length=0.034 radius=0.074792; visual mesh filename=package://pr2_description/meshes/base_v0/wheel.dae
- link head_pan_link: mass 1.611118 -> 6.339; geometry collision mesh filename=package://pr2_description/meshes/head_v0/head_pan_L.stl; visual mesh filename=package://pr2_description/meshes/head_v0/head_pan.dae
- link head_tilt_link: mass 1.749727 -> 4.479; geometry collision mesh filename=package://pr2_description/meshes/head_v0/head_tilt_L.stl; visual mesh filename=package://pr2_description/meshes/head_v0/head_tilt.dae
- link high_def_frame: geometry visual box size=0.04 0.04 0.04
- link high_def_optical_frame: geometry visual cylinder length=0.05 radius=0.02
- link l_elbow_flex_link: geometry collision mesh filename=package://pr2_description/meshes/upper_arm_v0/elbow_flex.stl; visual mesh filename=package://pr2_description/meshes/upper_arm_v0/elbow_flex.dae
- link l_forearm_cam_frame: geometry visual box size=0.01 0.01 0.01
- link l_forearm_link: geometry collision mesh filename=package://pr2_description/meshes/forearm_v0/forearm.stl; visual mesh filename=package://pr2_description/meshes/forearm_v0/forearm.dae
- link l_gripper_l_finger_link: geometry collision mesh filename=package://pr2_description/meshes/gripper_v0/l_finger.stl; visual mesh filename=package://pr2_description/meshes/gripper_v0/l_finger.dae
- link l_gripper_l_finger_tip_link: geometry collision mesh filename=package://pr2_description/meshes/gripper_v0/l_finger_tip.stl; visual mesh filename=package://pr2_description/meshes/gripper_v0/l_finger_tip.dae
- link l_gripper_palm_link: geometry collision mesh filename=package://pr2_description/meshes/gripper_v0/gripper_palm.stl; visual mesh filename=package://pr2_description/meshes/gripper_v0/gripper_palm.dae
- link l_gripper_r_finger_link: geometry collision mesh filename=package://pr2_description/meshes/gripper_v0/l_finger.stl; visual mesh filename=package://pr2_description/meshes/gripper_v0/l_finger.dae
- link l_gripper_r_finger_tip_link: geometry collision mesh filename=package://pr2_description/meshes/gripper_v0/l_finger_tip.stl; visual mesh filename=package://pr2_description/meshes/gripper_v0/l_finger_tip.dae
- link l_shoulder_pan_link: geometry collision mesh filename=package://pr2_description/meshes/shoulder_v0/shoulder_pan.s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; visual mesh filename=package://pr2_description/meshes/shoulder_v0/shoulder_pan.d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
- link l_upper_arm_link: geometry collision mesh filename=package://pr2_description/meshes/upper_arm_v0/upper_arm.stl; visual mesh filename=package://pr2_description/meshes/upper_arm_v0/upper_arm.dae
- link l_wrist_flex_link: geometry collision mesh filename=package://pr2_description/meshes/forearm_v0/wrist_flex.stl; visual mesh filename=package://pr2_description/meshes/forearm_v0/wrist_flex.dae
- link narrow_stereo_gazebo_l_stereo_camera_frame: geometry visual box size=0.01 0.01 0.01
- link narrow_stereo_gazebo_r_stereo_camera_frame: geometry visual box size=0.01 0.01 0.01
- link r_elbow_flex_link: geometry collision mesh filename=package://pr2_description/meshes/upper_arm_v0/elbow_flex.stl; visual mesh filename=package://pr2_description/meshes/upper_arm_v0/elbow_flex.dae
- link r_forearm_cam_frame: geometry visual box size=0.01 0.01 0.01
- link r_forearm_link: geometry collision mesh filename=package://pr2_description/meshes/forearm_v0/forearm.stl; visual mesh filename=package://pr2_description/meshes/forearm_v0/forearm.dae
- link r_gripper_l_finger_link: geometry collision mesh filename=package://pr2_description/meshes/gripper_v0/l_finger.stl; visual mesh filename=package://pr2_description/meshes/gripper_v0/l_finger.dae
- link r_gripper_l_finger_tip_link: geometry collision mesh filename=package://pr2_description/meshes/gripper_v0/l_finger_tip.stl; visual mesh filename=package://pr2_description/meshes/gripper_v0/l_finger_tip.dae
- link r_gripper_palm_link: geometry collision mesh filename=package://pr2_description/meshes/gripper_v0/gripper_palm.stl; visual mesh filename=package://pr2_description/meshes/gripper_v0/gripper_palm.dae
- link r_gripper_r_finger_link: geometry collision mesh filename=package://pr2_description/meshes/gripper_v0/l_finger.stl; visual mesh filename=package://pr2_description/meshes/gripper_v0/l_finger.dae
- link r_gripper_r_finger_tip_link: geometry collision mesh filename=package://pr2_description/meshes/gripper_v0/l_finger_tip.stl; visual mesh filename=package://pr2_description/meshes/gripper_v0/l_finger_tip.dae
- link r_shoulder_pan_link: geometry collision mesh filename=package://pr2_description/meshes/shoulder_v0/shoulder_pan.s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; visual mesh filename=package://pr2_description/meshes/shoulder_v0/shoulder_pan.d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
- link r_upper_arm_link: geometry collision mesh filename=package://pr2_description/meshes/upper_arm_v0/upper_arm.stl; visual mesh filename=package://pr2_description/meshes/upper_arm_v0/upper_arm.dae
- link r_wrist_flex_link: geometry collision mesh filename=package://pr2_description/meshes/forearm_v0/wrist_flex.stl; visual mesh filename=package://pr2_description/meshes/forearm_v0/wrist_flex.dae
- link torso_lift_link: geometry collision mesh filename=package://pr2_description/meshes/torso_v0/torso_lift_L.stl; visual mesh filename=package://pr2_description/meshes/torso_v0/torso_lift.dae
- link wide_stereo_gazebo_l_stereo_camera_frame: geometry visual box size=0.01 0.01 0.01
- link wide_stereo_gazebo_r_stereo_camera_frame: geometry visual box size=0.01 0.01 0.01
Joints:
- removed joint l_gripper_l_parallel_root_joint
- removed joint l_gripper_r_parallel_root_joint
- removed joint r_gripper_l_parallel_root_joint
- removed joint r_gripper_r_parallel_root_joint
- added joint base_bellow_joint: type fixed, parent base_link, child base_bellow_link, origin xyz=-0.29 0 0.8 rpy=0 0 0
- added joint l_torso_lift_side_plate_joint: type fixed, parent torso_lift_link, child l_torso_lift_side_plate_link, origin xyz=0.0535 -0.209285 0.176625
- added joint projector_wg6802418_child_frame_joint: type fixed, parent projector_wg6802418_frame, child projector_wg6802418_child_frame, origin xyz=0 0 0 rpy=0 -1.57079632679 0
- added joint projector_wg6802418_frame_joint: type fixed, parent head_plate_frame, child projector_wg6802418_frame, origin xyz=0 0.109 0.035 rpy=0 0 0
- added joint r_torso_lift_side_plate_joint: type fixed, parent torso_lift_link, child r_torso_lift_side_plate_link, origin xyz=0.0535  0.209285 0.176625
- joint l_gripper_joint: child (none) -> l_gripper_l_finger_tip_frame; parent (none) -> l_gripper_r_finger_tip_link
- joint l_wrist_flex_joint: limit lower=-2.094 upper=0.0 effort=10 velocity=3.078 -> lower=-2.18 upper=0.0 effort=10 velocity=3.078
- joint r_gripper_joint: child (none) -> r_gripper_l_finger_tip_frame; parent (none) -> r_gripper_r_finger_tip_link
- joint r_wrist_flex_joint: limit lower=-2.094 upper=0.0 effort=10 velocity=3.078 -> lower=-2.18 upper=0.0 effort=10 velocity=3.078

Commit message: Clean up code and get regression tests working

File: robot_state_publisher/test/pr2.urdf (robot description, URDF)
Before this commit: robot pr2, 80 links, 81 joints
Links:
- removed link l_gripper_l_parallel_link
- removed link l_gripper_r_parallel_link
- removed link r_gripper_l_parallel_link
- removed link r_gripper_r_parallel_link
- added link base_bellow_link, mass 1.0; collision box size=0.05 0.37 0.3; visual box size=0.05 0.37 0.3
- added link l_gripper_l_finger_tip_frame
- added link l_torso_lift_side_plate_link, mass 0.1
- added link projector_wg6802418_child_frame, mass 0.01; visual cylinder length=0.05 radius=0.02
- added link projector_wg6802418_frame, mass 0.01; visual box size=0.04 0.04 0.04
- added link r_gripper_l_finger_tip_frame
- added link r_torso_lift_side_plate_link, mass 0.1
- link base_laser_link: geometry 
- link base_link: geometry collision mesh filename=package://pr2_description/meshes/base_v0/base_L.stl; visual mesh filename=package://pr2_description/meshes/base_v0/base.dae
- link bl_caster_l_wheel_link: geometry collision cylinder length=0.034 radius=0.074792; visual mesh filename=package://pr2_description/meshes/base_v0/wheel.dae
- link bl_caster_r_wheel_link: geometry collision cylinder length=0.034 radius=0.074792; visual mesh filename=package://pr2_description/meshes/base_v0/wheel.dae
- link br_caster_l_wheel_link: geometry collision cylinder length=0.034 radius=0.074792; visual mesh filename=package://pr2_description/meshes/base_v0/wheel.dae
- link br_caster_r_wheel_link: geometry collision cylinder length=0.034 radius=0.074792; visual mesh filename=package://pr2_description/meshes/base_v0/wheel.dae
- link double_stereo_link: geometry visual box size=0.02 0.12 0.05
- link fl_caster_l_wheel_link: geometry collision cylinder length=0.034 radius=0.074792; visual mesh filename=package://pr2_description/meshes/base_v0/wheel.dae
- link fl_caster_r_wheel_link: geometry collision cylinder length=0.034 radius=0.074792; visual mesh filename=package://pr2_description/meshes/base_v0/wheel.dae
- link fr_caster_l_wheel_link: geometry collision cylinder length=0.034 radius=0.074792; visual mesh filename=package://pr2_description/meshes/base_v0/wheel.dae
- link fr_caster_r_wheel_link: geometry collision cylinder length=0.034 radius=0.074792; visual mesh filename=package://pr2_description/meshes/base_v0/wheel.dae
- link head_pan_link: mass 1.611118 -> 6.339; geometry collision mesh filename=package://pr2_description/meshes/head_v0/head_pan_L.stl; visual mesh filename=package://pr2_description/meshes/head_v0/head_pan.dae
- link head_tilt_link: mass 1.749727 -> 4.479; geometry collision mesh filename=package://pr2_description/meshes/head_v0/head_tilt_L.stl; visual mesh filename=package://pr2_description/meshes/head_v0/head_tilt.dae
- link high_def_frame: geometry visual box size=0.04 0.04 0.04
- link high_def_optical_frame: geometry visual cylinder length=0.05 radius=0.02
- link imu_link: geometry 
- link l_elbow_flex_link: geometry collision mesh filename=package://pr2_description/meshes/upper_arm_v0/elbow_flex.stl; visual mesh filename=package://pr2_description/meshes/upper_arm_v0/elbow_flex.dae
- link l_forearm_cam_frame: geometry 
- link l_forearm_link: geometry collision mesh filename=package://pr2_description/meshes/forearm_v0/forearm.stl; visual mesh filename=package://pr2_description/meshes/forearm_v0/forearm.dae
- link l_gripper_l_finger_link: geometry collision mesh filename=package://pr2_description/meshes/gripper_v0/l_finger.stl; visual mesh filename=package://pr2_description/meshes/gripper_v0/l_finger.dae
- link l_gripper_l_finger_tip_link: geometry collision mesh filename=package://pr2_description/meshes/gripper_v0/l_finger_tip.stl; visual mesh filename=package://pr2_description/meshes/gripper_v0/l_finger_tip.dae
- link l_gripper_palm_link: geometry collision mesh filename=package://pr2_description/meshes/gripper_v0/gripper_palm.stl; visual mesh filename=package://pr2_description/meshes/gripper_v0/gripper_palm.dae
- link l_gripper_r_finger_link: geometry collision mesh filename=package://pr2_description/meshes/gripper_v0/l_finger.stl; visual mesh filename=package://pr2_description/meshes/gripper_v0/l_finger.dae
- link l_gripper_r_finger_tip_link: geometry collision mesh filename=package://pr2_description/meshes/gripper_v0/l_finger_tip.stl; visual mesh filename=package://pr2_description/meshes/gripper_v0/l_finger_tip.dae
- link l_shoulder_pan_link: geometry collision mesh filename=package://pr2_description/meshes/shoulder_v0/shoulder_pan.s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; visual mesh filename=package://pr2_description/meshes/shoulder_v0/shoulder_pan.d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
- link l_upper_arm_link: geometry collision mesh filename=package://pr2_description/meshes/upper_arm_v0/upper_arm.stl; visual mesh filename=package://pr2_description/meshes/upper_arm_v0/upper_arm.dae
- link l_wrist_flex_link: geometry collision mesh filename=package://pr2_description/meshes/forearm_v0/wrist_flex.stl; visual mesh filename=package://pr2_description/meshes/forearm_v0/wrist_flex.dae
- link laser_tilt_link: geometry 
- link narrow_stereo_gazebo_l_stereo_camera_frame: geometry 
- link narrow_stereo_gazebo_r_stereo_camera_frame: geometry 
- link narrow_stereo_link: geometry 
- link r_elbow_flex_link: geometry collision mesh filename=package://pr2_description/meshes/upper_arm_v0/elbow_flex.stl; visual mesh filename=package://pr2_description/meshes/upper_arm_v0/elbow_flex.dae
- link r_forearm_cam_frame: geometry 
- link r_forearm_link: geometry collision mesh filename=package://pr2_description/meshes/forearm_v0/forearm.stl; visual mesh filename=package://pr2_description/meshes/forearm_v0/forearm.dae
- link r_gripper_l_finger_link: geometry collision mesh filename=package://pr2_description/meshes/gripper_v0/l_finger.stl; visual mesh filename=package://pr2_description/meshes/gripper_v0/l_finger.dae
- link r_gripper_l_finger_tip_link: geometry collision mesh filename=package://pr2_description/meshes/gripper_v0/l_finger_tip.stl; visual mesh filename=package://pr2_description/meshes/gripper_v0/l_finger_tip.dae
- link r_gripper_palm_link: geometry collision mesh filename=package://pr2_description/meshes/gripper_v0/gripper_palm.stl; visual mesh filename=package://pr2_description/meshes/gripper_v0/gripper_palm.dae
- link r_gripper_r_finger_link: geometry collision mesh filename=package://pr2_description/meshes/gripper_v0/l_finger.stl; visual mesh filename=package://pr2_description/meshes/gripper_v0/l_finger.dae
- link r_gripper_r_finger_tip_link: geometry collision mesh filename=package://pr2_description/meshes/gripper_v0/l_finger_tip.stl; visual mesh filename=package://pr2_description/meshes/gripper_v0/l_finger_tip.dae
- link r_shoulder_pan_link: geometry collision mesh filename=package://pr2_description/meshes/shoulder_v0/shoulder_pan.s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; visual mesh filename=package://pr2_description/meshes/shoulder_v0/shoulder_pan.d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
- link r_upper_arm_link: geometry collision mesh filename=package://pr2_description/meshes/upper_arm_v0/upper_arm.stl; visual mesh filename=package://pr2_description/meshes/upper_arm_v0/upper_arm.dae
- link r_wrist_flex_link: geometry collision mesh filename=package://pr2_description/meshes/forearm_v0/wrist_flex.stl; visual mesh filename=package://pr2_description/meshes/forearm_v0/wrist_flex.dae
- link sensor_mount_link: geometry visual box size=0.01 0.01 0.01
- link torso_lift_link: geometry collision mesh filename=package://pr2_description/meshes/torso_v0/torso_lift_L.stl; visual mesh filename=package://pr2_description/meshes/torso_v0/torso_lift.dae
- link wide_stereo_gazebo_l_stereo_camera_frame: geometry 
- link wide_stereo_gazebo_r_stereo_camera_frame: geometry 
- link wide_stereo_link: geometry 
Joints:
- removed joint l_gripper_l_parallel_root_joint
- removed joint l_gripper_r_parallel_root_joint
- removed joint r_gripper_l_parallel_root_joint
- removed joint r_gripper_r_parallel_root_joint
- added joint base_bellow_joint: type fixed, parent base_link, child base_bellow_link, origin xyz=-0.29 0 0.8 rpy=0 0 0
- added joint l_torso_lift_side_plate_joint: type fixed, parent torso_lift_link, child l_torso_lift_side_plate_link, origin xyz=0.0535 -0.209285 0.176625
- added joint projector_wg6802418_child_frame_joint: type fixed, parent projector_wg6802418_frame, child projector_wg6802418_child_frame, origin xyz=0 0 0 rpy=0 -1.57079632679 0
- added joint projector_wg6802418_frame_joint: type fixed, parent head_plate_frame, child projector_wg6802418_frame, origin xyz=0 0.109 0.035 rpy=0 0 0
- added joint r_torso_lift_side_plate_joint: type fixed, parent torso_lift_link, child r_torso_lift_side_plate_link, origin xyz=0.0535  0.209285 0.176625
- joint l_gripper_joint: child (none) -> l_gripper_l_finger_tip_frame; parent (none) -> l_gripper_r_finger_tip_link
- joint l_wrist_flex_joint: limit lower=-2.094 upper=0.0 effort=10 velocity=3.078 -> lower=-2.18 upper=0.0 effort=10 velocity=3.078
- joint r_gripper_joint: child (none) -> r_gripper_l_finger_tip_frame; parent (none) -> r_gripper_r_finger_tip_link
- joint r_wrist_flex_joint: limit lower=-2.094 upper=0.0 effort=10 velocity=3.078 -> lower=-2.18 upper=0.0 effort=10 velocity=3.078
